File: kicad/cocousbhost.kicad_sch (KiCad schematic)
At the start: 31 parts, among them J1 Conn_01x03_Male, J2 Jumper_2_Bridged, J3 USB_A, Q1 2N2222, SW1 SW_DIP_x07, U1 74LS30, U2 Coco_Cart_Connector, U3 74LS682, U4 74LS04, U5 74LS74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

Commit message: Renamed to CoCo USB Host
Other:
- title: CoCo USB Pak -> CoCo USB Host
Changed lines of the file:
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@@
 	(paper "A4")
 	(title_block
-		(title "CoCo USB Pak")
+		(title "CoCo USB Host")
 		(company "Don Barber")
-		(comment 1 "https://github.com/barberd/cocousbpak")
+		(comment 1 "https://github.com/barberd/cocousbhost")
 		(comment 2 "Licensed GPL v3")
 	)
